File: hardware/ide.kicad_sch (KiCad schematic)
At the start: 13 parts, among them J5 IDE, U2 SN74CB3T3245PWR, U3 SN74CB3T3245PWR, U5 SN74CB3T3245PWR, U6 SN74CB3T3245PWR

Commit message: PCB rev 0.2: RP2350B on the board instead of the PGA2350 module
The PGA2350 is replaced by an RP2350B with Raspberry Pi's minimal-design
support circuit: their core regulator (polarity-marked inductor), 12 MHz
crystal, W25Q128 flash and USB 27R, with their regulator, QSPI and USB
layout copied relative to the VREG_LX pin; an AMS1117 makes 3V3. GPIO
numbers are unchanged. Supply pins each have a via under the chip.

Cheaper parts from the HDD Synth Mk5: HRO TYPE-C-31-M-12 USB-C, TS-1187A
buttons, and a generic TF PUSH microSD socket. The CB3T3245 bus switches
stay. Every symbol carries its LCSC part number, and Fabrication Toolkit
offsets where JLCPCB's footprint differs from KiCad's; jlcpcb.py applies
the same fitted corrections. check_netlist.py also checks the RP2350
support circuit. ERC and DRC are clean; parts for 5 boards about $68.50.

Co-Authored-By: Claude Opus 5.5 <noreply@anthropic.com>
Parts:
- C4, C5, C7, C8: LCSC (none) -> C14663
- J5: FT Rotation Offset (none) -> -90; LCSC (none) -> C19193815
- R13: LCSC (none) -> C25804
- R14, R15: LCSC (none) -> C23140
- U2, U3, U5, U6: LCSC (none) -> C15298
Other:
- note added: "33 R damping on the strobes, close to the RP2350."
- note added: "IDE bus through four SN74CB3T3245 FET bus switches: A side to the RP2350, B side to the IDE header. OE# low = connected. They cap what the RP2350 sees at about 3.3 V and isolate it when unpowered (Ioff). No pull-ups or pull-downs on the bus: the host provides them. IORDY stays open drain."
- note removed: "33 R damping on the strobes, close to the PGA2350."
- note removed: "IDE bus through four SN74CB3T3245 FET bus switches: A side to the PGA2350, B side to the IDE header. OE# low = connected. They cap what the RP2350 sees at about 3.3 V and isolate it when unpowered (Ioff). No pull-ups or pull-downs on the bus: the host provides them. IORDY stays open drain."
